File: Hardware/PWMBoard.kicad_sch (KiCad schematic)
At the start: 27 parts, among them J1 Screw_Terminal_01x03, J2 Screw_Terminal_01x02, J3 AVR-ISP-6, Q1 IRF540N, Q2 IRF540N, Q3 IRF9540N, Q4 IRF9540N, Q5 BC547, Q6 BC547, U1 ATtiny2313-20P, U2 LM7805_TO220

Commit message: Update PCB
Parts:
- removed D4: D_Schottky, Diode_THT:D_5KP_P12.70mm_Horizontal, symbol Device:D_Schottky
- removed J1: Screw_Terminal_01x03, TerminalBlock_Phoenix:TerminalBlock_Phoenix_MKDS-3-3-5.08_1x03_P5.08mm_Horizontal, symbol Connector:Screw_Terminal_01x03
- added C3, C4: 10uF, Capacitor_THT:C_Disc_D8.0mm_W2.5mm_P5.00mm, symbol Device:C
- added D2: 4.7V, Diode_THT:D_T-1_P5.08mm_Horizontal, symbol Device:D_Zener
- added D3, D4: 12V, Diode_THT:D_A-405_P5.08mm_Vertical_KathodeUp, symbol Device:D_Zener
- added D5: 5V1, Diode_THT:D_A-405_P7.62mm_Horizontal, symbol Device:D_Zener
- added H1, H2, H3, H4: MountingHole, MountingHole:MountingHole_3.2mm_M3_DIN965, symbol Mechanical:MountingHole
- added J1, J4: Screw_Terminal_01x02, TerminalBlock_Phoenix:TerminalBlock_Phoenix_MKDS-3-2-5.08_1x02_P5.08mm_Horizontal, symbol Connector:Screw_Terminal_01x02
- added R12, R14: 10k, Resistor_THT:R_Axial_DIN0207_L6.3mm_D2.5mm_P5.08mm_Vertical, symbol Device:R
- Q1, Q2, Q3, Q4, U2: footprint Package_TO_SOT_THT:TO-220-3_Vertical -> Package_TO_SOT_THT:TO-220-3_Horizontal_TabDown
- R1, R3: footprint Resistor_THT:R_Axial_DIN0207_L6.3mm_D2.5mm_P2.54mm_Vertical -> Resistor_THT:R_Axial_DIN0207_L6.3mm_D2.5mm_P5.08mm_Vertical
- R10: footprint Resistor_THT:R_Axial_DIN0207_L6.3mm_D2.5mm_P7.62mm_Horizontal -> Resistor_THT:R_Axial_DIN0207_L6.3mm_D2.5mm_P5.08mm_Vertical
- R11, R9: footprint Resistor_THT:R_Axial_DIN0207_L6.3mm_D2.5mm_P7.62mm_Horizontal -> Resistor_THT:R_Axial_DIN0207_L6.3mm_D2.5mm_P2.54mm_Vertical
- R13: value 100k -> 10k
- R4: footprint Resistor_THT:R_Axial_DIN0207_L6.3mm_D2.5mm_P5.08mm_Vertical -> Resistor_THT:R_Axial_DIN0207_L6.3mm_D2.5mm_P10.16mm_Horizontal
- R5: value 2.2k -> 10k
- R7: value 2.2k -> 10k; footprint Resistor_THT:R_Axial_DIN0207_L6.3mm_D2.5mm_P5.08mm_Vertical -> Resistor_THT:R_Axial_DIN0207_L6.3mm_D2.5mm_P10.16mm_Horizontal
Connections:
- net down is gone; now on net A: R11.1
- net +5V: now also C3.1, D5.1 (K)
- net A: now also J4.2 (Pin_2); no longer J2.1 (Pin_1), Q1.2 (D), Q4.3 (S)
- net AH: now also D4.2 (A)
- net B: now also J4.1 (Pin_1), R14.1; no longer J2.2 (Pin_2), Q2.2 (D), Q3.3 (S)
- net BH: now also D3.2 (A)
- net GND: now also C3.2, C4.2, D2.2 (A), D5.2 (A), J1.1 (Pin_1), R12.2
- net VCC: now also Q3.3 (S), Q4.3 (S), C4.1, D3.1 (K), D4.1 (K), J1.2 (Pin_2); no longer Q3.2 (D), Q4.2 (D)
- net cAH: now also U1.15 (PB3); no longer U1.14 (PB2)
- net cAL: now also U1.13 (PB1); no longer U1.12 (PB0)
- net cBH: now also U1.16 (PB4); no longer U1.13 (PB1)
- net cBL: now also U1.14 (PB2); no longer U1.15 (PB3)
- net cDown: no longer D1.1 (K), R11.2, R13.1
- net b: now reaches U1.4 (PA1/XTAL2)
- net b: now also D2.1 (K), R12.1, R14.2
- net a: now reaches U1.5 (PA0/XTAL1)
- net a: now also D1.1 (K), R11.2, R13.1
- new net motorA: J2.1 (Pin_1), Q1.2 (D), Q4.2 (D)
- new net motorB: J2.2 (Pin_2), Q2.2 (D), Q3.2 (D)
- no-connect marks 2 -> 0
Other:
- moved on the sheet: C1, C2, D1, R11, R13, U2
